Commit message: x-axis front

File: robots/quadruped.urdf (robot description, URDF)
Before this commit: robot quadruped, 52 links, 51 joints
Links:
- link pelvis: geometry collision box size=2.0 1.2 0.5; visual box size=2.0 1.2 0.5
Joints:
- joint backward_left_knee_joint: axis 1 0 0 -> 0 1 0; limit lower=-0.698131700798 upper=2.61799387799 effort=300 velocity=0.1 -> lower=-2.61799387799 upper=0.698131700798 effort=300 velocity=0.1; origin xyz=0 0 -0.41 rpy=-1.308996939 0 0 -> xyz=0 0 -0.41 rpy=0 1.308996939 0
- joint backward_left_thigh_pitch_joint: axis 1 0 0 -> 0 1 0; limit lower=-1.0471975512 upper=1.0471975512 effort=300 velocity=0.1 -> lower=-1.5707963268 upper=0.523598775598 effort=300 velocity=0.1; origin xyz=0 0 -0.095 rpy=0.523598775598 0 0 -> xyz=0 0 -0.095 rpy=0 -0.523598775598 0
- joint backward_left_thigh_roll_joint: axis 0 1 0 -> 1 0 0; origin xyz=-0.68 -0.7 -0.1 -> xyz=-0.7 0.68 -0.1
- joint backward_right_knee_joint: axis 1 0 0 -> 0 1 0; limit lower=-0.698131700798 upper=2.61799387799 effort=300 velocity=0.1 -> lower=-2.61799387799 upper=0.698131700798 effort=300 velocity=0.1; origin xyz=0 0 -0.41 rpy=-1.308996939 0 0 -> xyz=0 0 -0.41 rpy=0 1.308996939 0
- joint backward_right_thigh_pitch_joint: axis 1 0 0 -> 0 1 0; limit lower=-1.0471975512 upper=1.0471975512 effort=300 velocity=0.1 -> lower=-1.5707963268 upper=0.523598775598 effort=300 velocity=0.1; origin xyz=0 0 -0.095 rpy=0.523598775598 0 0 -> xyz=0 0 -0.095 rpy=0 -0.523598775598 0
- joint backward_right_thigh_roll_joint: axis 0 1 0 -> 1 0 0; origin xyz=0.68 -0.7 -0.1 -> xyz=-0.7 -0.68 -0.1
- joint forward_left_knee_joint: axis 1 0 0 -> 0 1 0; limit lower=-2.61799387799 upper=0.698131700798 effort=300 velocity=0.1 -> lower=-0.698131700798 upper=2.61799387799 effort=300 velocity=0.1; origin xyz=0 0 -0.41 rpy=1.308996939 0 0 -> xyz=0 0 -0.41 rpy=0 -1.308996939 0
- joint forward_left_thigh_pitch_joint: axis 1 0 0 -> 0 1 0; limit lower=-1.0471975512 upper=1.0471975512 effort=300 velocity=0.1 -> lower=-1.5707963268 upper=0.523598775598 effort=300 velocity=0.1; origin xyz=0 0 -0.095 rpy=-0.523598775598 0 0 -> xyz=0 0 -0.095 rpy=0 0.523598775598 0
- joint forward_left_thigh_roll_joint: axis 0 1 0 -> 1 0 0; origin xyz=-0.68 0.7 -0.1 -> xyz=0.7 0.68 -0.1
- joint forward_right_knee_joint: axis 1 0 0 -> 0 1 0; limit lower=-2.61799387799 upper=0.698131700798 effort=300 velocity=0.1 -> lower=-0.698131700798 upper=2.61799387799 effort=300 velocity=0.1; origin xyz=0 0 -0.41 rpy=1.308996939 0 0 -> xyz=0 0 -0.41 rpy=0 -1.308996939 0
- joint forward_right_thigh_pitch_joint: axis 1 0 0 -> 0 1 0; limit lower=-1.0471975512 upper=1.0471975512 effort=300 velocity=0.1 -> lower=-1.5707963268 upper=0.523598775598 effort=300 velocity=0.1; origin xyz=0 0 -0.095 rpy=-0.523598775598 0 0 -> xyz=0 0 -0.095 rpy=0 0.523598775598 0
- joint forward_right_thigh_roll_joint: axis 0 1 0 -> 1 0 0; origin xyz=0.68 0.7 -0.1 -> xyz=0.7 -0.68 -0.1
- joint pelvis_shoulder_fixed_joint: origin xyz=0 0.8 0.4 -> xyz=0.8 0 0.4

File: urdfs/common.xacro (robot description, xacro)
@@ -46,6 +46,6 @@
 <xacro:property name="thigh_roll_min" value="15"/>
 <xacro:property name="thigh_roll_max" value="60"/>
-<xacro:property name="thigh_pitch_min" value="-60"/>
-<xacro:property name="thigh_pitch_max" value="60"/>
+<xacro:property name="thigh_pitch_min" value="-90"/>
+<xacro:property name="thigh_pitch_max" value="30"/>
 <xacro:property name="knee_pitch_min" value="40"/>
 <xacro:property name="knee_pitch_max" value="150"/>

File: urdfs/leg/leg.urdf.xacro (robot description, xacro)
@@ -9,8 +9,8 @@
    <!-- joint between the thigh_roll_cylinder and pelvic -->
     <joint name="${prefix}_thigh_roll_joint" type="revolute">
-      <origin xyz="${reflect_lateral*(pelvis_w/2+thigh_r_r)} ${reflect_fb*(pelvis_l/2-0.3)} -0.1"/>    <!-- 0.3 and 0.1 are the offset provided for the thigh_roll_cylinder from the front and centerline below-->
+      <origin xyz="${reflect_fb*(pelvis_l/2-0.3)} ${-reflect_lateral*(pelvis_w/2+thigh_r_r)} -0.1"/>    <!-- 0.3 and 0.1 are the offset provided for the thigh_roll_cylinder from the front and centerline below-->
       <parent link ="pelvis"/>
       <child link="${prefix}_thigh_roll_cylinder"/>
-      <axis xyz="0 1 0"/>
+      <axis xyz="1 0 0"/>
       <limit effort="${joint_limit_effort}" velocity="${joint_velocity}"
       lower="${-(1-left_right)*thigh_roll_min*PI/180-left_right*thigh_roll_max*PI/180}"
@@ -26,8 +26,8 @@
     <!-- the joint which allows the pitch motion of the thigh -->
     <joint name="${prefix}_thigh_pitch_joint" type="revolute">
-      <origin xyz="0 0 -${thigh_p_r+thigh_bwn_l/2}" rpy="${-30*front_back*deg_to_rad} 0 0"/>
+      <origin xyz="0 0 -${thigh_p_r+thigh_bwn_l/2}" rpy="0 ${30*front_back*deg_to_rad} 0"/>
       <parent link="${prefix}_thigh_bwn_cylinder"/>
       <child link="${prefix}_thigh_pitch_cylinder"/>
-      <axis xyz="1 0 0"/>
+      <axis xyz="0 1 0"/>
       <limit effort="${joint_limit_effort}" velocity="${joint_velocity}" lower="${thigh_pitch_min*PI/180}" upper="${thigh_pitch_max*PI/180}"/>
       <dynamics damping="0.1" friction="0" />
@@ -41,10 +41,10 @@
     <!-- knee joint -->
     <joint name="${prefix}_knee_joint" type="revolute">
-      <origin xyz="0 0 -${knee_r+upper_leg_l/2}" rpy="${75*front_back*deg_to_rad} 0 0"/>
+      <origin xyz="0 0 -${knee_r+upper_leg_l/2}" rpy="0 ${-75*front_back*deg_to_rad} 0"/>
       <parent link="${prefix}_upper_leg"/>
       <child link="${prefix}_knee_cylinder"/>
-      <axis xyz="1 0 0"/>
-      <limit effort="${joint_limit_effort}" velocity="${joint_velocity}" lower="${(-(1+front_back)/2*knee_pitch_max-(1-front_back)/2*knee_pitch_min)*PI/180}"
-				         upper="${((1+front_back)/2*knee_pitch_min+(1-front_back)/2*knee_pitch_max)*PI/180}"/>
+      <axis xyz="0 1 0"/>
+      <limit effort="${joint_limit_effort}" velocity="${joint_velocity}" lower="${(-(1+front_back)/2*knee_pitch_min-(1-front_back)/2*knee_pitch_max)*PI/180}"
+				         upper="${((1+front_back)/2*knee_pitch_max+(1-front_back)/2*knee_pitch_min)*PI/180}"/>
       <dynamics damping="0.1" friction="0" />
     </joint>
@@ -75,9 +75,9 @@
           <cylinder radius="${thigh_r_r}" length="${thigh_r_l}"/>
         </geometry>
-        <origin xyz="0 0 0" rpy="${PI_2} 0 0"/>
-        <material name="red"/>
-      </visual>
-      <collision>
-				<origin xyz="0 0 0" rpy="${PI_2} 0 0"/>
+        <origin xyz="0 0 0" rpy="0 ${PI_2} 0"/>
+        <material name="red"/>
+      </visual>
+      <collision>
+				<origin xyz="0 0 0" rpy="0 ${PI_2} 0"/>
         <geometry>
           <cylinder radius="${thigh_r_r}" length="${thigh_r_l}"/>
@@ -120,9 +120,9 @@
           <cylinder radius="${thigh_p_r}" length="${thigh_p_l}"/>
         </geometry>
-        <origin xyz="0 0 0" rpy="0 ${PI_2} 0"/>
-        <material name="red"/>
-      </visual>
-      <collision>
-				<origin xyz="0 0 0" rpy="0 ${PI_2} 0"/>
+        <origin xyz="0 0 0" rpy="${PI_2} 0 0"/>
+        <material name="red"/>
+      </visual>
+      <collision>
+				<origin xyz="0 0 0" rpy="${PI_2} 0 0"/>
         <geometry>
           <cylinder radius="${thigh_p_r}" length="${thigh_p_l}"/>
@@ -165,9 +165,9 @@
           <cylinder radius="${knee_r}" length="${knee_l}"/>
         </geometry>
-        <origin xyz="0 0 0" rpy="0 ${PI_2} 0"/>
-        <material name="red"/>
-      </visual>
-      <collision>
-				<origin xyz="0 0 0" rpy="0 ${PI_2} 0"/>
+        <origin xyz="0 0 0" rpy="${PI_2} 0 0"/>
+        <material name="red"/>
+      </visual>
+      <collision>
+				<origin xyz="0 0 0" rpy="${PI_2} 0 0"/>
         <geometry>
           <cylinder radius="${knee_r}" length="${knee_l}"/>

File: urdfs/torso/torso.urdf.xacro (robot description, xacro)
@@ -8,5 +8,5 @@
 		<!-- Joints -->
 		<joint name="pelvis_shoulder_fixed_joint" type="fixed">
-			<origin xyz="0 ${pelvis_l/2-0.2} ${spine_l/2+pelvis_h/2}" />
+			<origin xyz="${pelvis_l/2-0.2} 0 ${spine_l/2+pelvis_h/2}" />
 			<parent link="pelvis"/>
 			<child link="spine_cylinder"/>

File: urdfs/trunk/trunk.urdf.xacro (robot description, xacro)
@@ -33,5 +33,5 @@
 			<visual>
 				<geometry>
-					<box size="${pelvis_w} ${pelvis_l} ${pelvis_h}"/>
+					<box size="${pelvis_l} ${pelvis_w} ${pelvis_h}"/>
 				</geometry>
 				<origin xyz="0 0 0" rpy="0 0 0"/>
@@ -40,5 +40,5 @@
 			<collision>
 				<geometry>
-					<box size="${pelvis_w} ${pelvis_l} ${pelvis_h}"/>
+					<box size="${pelvis_l} ${pelvis_w} ${pelvis_h}"/>
 				</geometry>
 			</collision>

Commit message: updating torso

File: robots/quadruped.urdf (robot description, URDF)
Before this commit: robot quadruped, 52 links, 51 joints
Joints:
- joint left_elbow_joint: type fixed -> revolute
- joint left_finger_joint1: type fixed -> revolute
- joint left_finger_joint2: type fixed -> revolute
- joint left_shoulder_pitch_joint: axis 1 0 0 -> 0 1 0; origin xyz=-0.65 0 0 -> xyz=0 -0.65 0; type fixed -> revolute
- joint left_shoulder_roll_joint: axis 0 1 0 -> 1 0 0; origin xyz=-0.15 0 0 rpy=0 0.3 0 -> xyz=0 -0.15 0 rpy=0 0.3 0; type fixed -> revolute
- joint left_shoulder_yaw_joint: type fixed -> revolute
- joint right_elbow_joint: type fixed -> revolute
- joint right_finger_joint1: type fixed -> revolute
- joint right_finger_joint2: type fixed -> revolute
- joint right_shoulder_pitch_joint: axis 1 0 0 -> 0 1 0; origin xyz=0.65 0 0 -> xyz=0 0.65 0; type fixed -> revolute
- joint right_shoulder_roll_joint: axis 0 1 0 -> 1 0 0; origin xyz=0.15 0 0 rpy=0 -0.3 0 -> xyz=0 0.15 0 rpy=0 -0.3 0; type fixed -> revolute
- joint right_shoulder_yaw_joint: type fixed -> revolute

File: urdfs/arm/arm.urdf.xacro (robot description, xacro)
@@ -6,16 +6,16 @@
 	<xacro:macro name="arm" params="prefix reflect">
   <!-- Joints -->
-  <joint name="${prefix}_shoulder_pitch_joint" type="fixed">
-    <origin xyz="${reflect*(shoulder_w/2+shoulder_pitch_l/2)} 0 0"/>
+  <joint name="${prefix}_shoulder_pitch_joint" type="revolute">
+    <origin xyz="0 ${reflect*(shoulder_w/2+shoulder_pitch_l/2)} 0"/>
     <parent link="shoulder"/>
     <child link="${prefix}_shoulder_pitch_cylinder"/>
-    <axis xyz="1 0 0"/>
-    <limit effort="${joint_limit_effort}" velocity="${joint_velocity}" lower="-3.14" upper="3.14"/>
-  </joint>
-	<joint name="${prefix}_shoulder_roll_joint" type="fixed">
-    <origin xyz="${reflect*(shoulder_roll_r+shoulder_pitch_l/2)} 0 0"  rpy="0 ${-reflect*0.3} 0"/>
+    <axis xyz="0 1 0"/>
+    <limit effort="${joint_limit_effort}" velocity="${joint_velocity}" lower="-3.14" upper="3.14"/>
+  </joint>
+	<joint name="${prefix}_shoulder_roll_joint" type="revolute">
+    <origin xyz="0 ${reflect*(shoulder_roll_r+shoulder_pitch_l/2)} 0"  rpy="0 ${-reflect*0.3} 0"/>
     <parent link="${prefix}_shoulder_pitch_cylinder"/>
     <child link="${prefix}_shoulder_roll_cylinder"/>
-    <axis xyz="0 1 0"/>
+    <axis xyz="1 0 0"/>
     <limit effort="${joint_limit_effort}" velocity="${joint_velocity}" lower="-3.14" upper="3.14"/>
   </joint>
@@ -25,5 +25,5 @@
     <child link="${prefix}_shoulder_bwn_cylinder"/>
   </joint>
-	<joint name="${prefix}_shoulder_yaw_joint" type="fixed">
+	<joint name="${prefix}_shoulder_yaw_joint" type="revolute">
     <origin xyz="0 0 -${shoulder_bwn_l/2+shoulder_yaw_l/2}"/>
     <parent link="${prefix}_shoulder_bwn_cylinder"/>
@@ -32,5 +32,5 @@
     <limit effort="${joint_limit_effort}" velocity="${joint_velocity}" lower="-3.14" upper="3.14"/>
   </joint>
-	<joint name="${prefix}_elbow_joint" type="fixed">
+	<joint name="${prefix}_elbow_joint" type="revolute">
     <origin xyz="0 0 -${elbow_r+shoulder_yaw_l/2}" rpy="0 ${reflect*0.3} 0"/>
     <parent link="${prefix}_shoulder_yaw_cylinder"/>
@@ -56,5 +56,5 @@
     <child link="${prefix}_gripper_fixed_link"/>
   </joint>
-	<joint name="${prefix}_finger_joint1" type="fixed">
+	<joint name="${prefix}_finger_joint1" type="revolute">
       <parent link="${prefix}_gripper_fixed_link"/>
       <child link="${prefix}_gripper_finger_link1"/>
@@ -63,5 +63,5 @@
       <limit effort="1" lower="-0.09" upper="0" velocity="1.0"/>
   </joint>
-	<joint name="${prefix}_finger_joint2" type="fixed">
+	<joint name="${prefix}_finger_joint2" type="revolute">
       <parent link="${prefix}_gripper_fixed_link"/>
       <child link="${prefix}_gripper_finger_link2"/>

Commit message: default direction toward x-axis version

File: robots/quadruped.urdf (robot description, URDF)
Before this commit: robot quadruped, 52 links, 51 joints
Links:
- link shoulder: geometry collision box size=0.5 1.2 0.3; visual box size=0.5 1.2 0.3
Joints:
- joint left_elbow_joint: axis 0 1 0 -> 1 0 0; origin xyz=0 0 -0.275 rpy=0 -0.3 0 -> xyz=0 0 -0.275 rpy=-0.3 0 0; type revolute -> fixed
- joint left_finger_joint1: type revolute -> fixed
- joint left_finger_joint2: type revolute -> fixed
- joint left_shoulder_pitch_joint: origin xyz=0 -0.65 0 -> xyz=0 0.65 0; type revolute -> fixed
- joint left_shoulder_roll_joint: origin xyz=0 -0.15 0 rpy=0 0.3 0 -> xyz=0 0.15 0 rpy=0.3 0 0; type revolute -> fixed
- joint left_shoulder_yaw_joint: type revolute -> fixed
- joint right_elbow_joint: axis 0 1 0 -> 1 0 0; origin xyz=0 0 -0.275 rpy=0 0.3 0 -> xyz=0 0 -0.275 rpy=0.3 0 0; type revolute -> fixed
- joint right_finger_joint1: type revolute -> fixed
- joint right_finger_joint2: type revolute -> fixed
- joint right_shoulder_pitch_joint: origin xyz=0 0.65 0 -> xyz=0 -0.65 0; type revolute -> fixed
- joint right_shoulder_roll_joint: origin xyz=0 0.15 0 rpy=0 -0.3 0 -> xyz=0 -0.15 0 rpy=-0.3 0 0; type revolute -> fixed
- joint right_shoulder_yaw_joint: type revolute -> fixed

File: robots/quadruped.urdf.xacro (robot description, xacro)
@@ -41,7 +41,7 @@
 	</xacro:quad_torso>
 	<!-- arm -->
-	<xacro:arm prefix="left" reflect="-1">
+	<xacro:arm prefix="left" reflect="1">
 	</xacro:arm>
-  <xacro:arm prefix="right" reflect="1">
+  <xacro:arm prefix="right" reflect="-1">
 	</xacro:arm>
 </robot>

File: urdfs/arm/arm.urdf.xacro (robot description, xacro)
@@ -6,5 +6,5 @@
 	<xacro:macro name="arm" params="prefix reflect">
   <!-- Joints -->
-  <joint name="${prefix}_shoulder_pitch_joint" type="revolute">
+  <joint name="${prefix}_shoulder_pitch_joint" type="fixed">
     <origin xyz="0 ${reflect*(shoulder_w/2+shoulder_pitch_l/2)} 0"/>
     <parent link="shoulder"/>
@@ -13,6 +13,6 @@
     <limit effort="${joint_limit_effort}" velocity="${joint_velocity}" lower="-3.14" upper="3.14"/>
   </joint>
-	<joint name="${prefix}_shoulder_roll_joint" type="revolute">
-    <origin xyz="0 ${reflect*(shoulder_roll_r+shoulder_pitch_l/2)} 0"  rpy="0 ${-reflect*0.3} 0"/>
+	<joint name="${prefix}_shoulder_roll_joint" type="fixed">
+    <origin xyz="0 ${reflect*(shoulder_roll_r+shoulder_pitch_l/2)} 0"  rpy="${reflect*0.3} 0 0"/>
     <parent link="${prefix}_shoulder_pitch_cylinder"/>
     <child link="${prefix}_shoulder_roll_cylinder"/>
@@ -25,5 +25,5 @@
     <child link="${prefix}_shoulder_bwn_cylinder"/>
   </joint>
-	<joint name="${prefix}_shoulder_yaw_joint" type="revolute">
+	<joint name="${prefix}_shoulder_yaw_joint" type="fixed">
     <origin xyz="0 0 -${shoulder_bwn_l/2+shoulder_yaw_l/2}"/>
     <parent link="${prefix}_shoulder_bwn_cylinder"/>
@@ -32,9 +32,9 @@
     <limit effort="${joint_limit_effort}" velocity="${joint_velocity}" lower="-3.14" upper="3.14"/>
   </joint>
-	<joint name="${prefix}_elbow_joint" type="revolute">
-    <origin xyz="0 0 -${elbow_r+shoulder_yaw_l/2}" rpy="0 ${reflect*0.3} 0"/>
+	<joint name="${prefix}_elbow_joint" type="fixed">
+    <origin xyz="0 0 -${elbow_r+shoulder_yaw_l/2}" rpy="${-reflect*0.3} 0 0"/>
     <parent link="${prefix}_shoulder_yaw_cylinder"/>
     <child link="${prefix}_elbow_cylinder"/>
-    <axis xyz="0 1 0"/>
+    <axis xyz="1 0 0"/>
     <limit effort="${joint_limit_effort}" velocity="${joint_velocity}" lower="-3.14" upper="3.14"/>
   </joint>
@@ -56,5 +56,5 @@
     <child link="${prefix}_gripper_fixed_link"/>
   </joint>
-	<joint name="${prefix}_finger_joint1" type="revolute">
+	<joint name="${prefix}_finger_joint1" type="fixed">
       <parent link="${prefix}_gripper_fixed_link"/>
       <child link="${prefix}_gripper_finger_link1"/>
@@ -63,5 +63,5 @@
       <limit effort="1" lower="-0.09" upper="0" velocity="1.0"/>
   </joint>
-	<joint name="${prefix}_finger_joint2" type="revolute">
+	<joint name="${prefix}_finger_joint2" type="fixed">
       <parent link="${prefix}_gripper_fixed_link"/>
       <child link="${prefix}_gripper_finger_link2"/>
@@ -76,4 +76,19 @@
         <cylinder radius="${shoulder_pitch_r}" length="${shoulder_pitch_l}"/>
       </geometry>
+      <origin xyz="0 0 0" rpy="${PI_2} 0 0"/>
+      <material name="red"/>
+    </visual>
+    <collision>
+			<origin xyz="0 0 0" rpy="${PI_2} 0 0"/>
+      <geometry>
+        <cylinder radius="${shoulder_pitch_r}" length="${shoulder_pitch_l}"/>
+      </geometry>
+    </collision>
+  </link>
+  <link name="${prefix}_shoulder_roll_cylinder">
+    <visual>
+      <geometry>
+        <cylinder radius="${shoulder_roll_r}" length="${shoulder_roll_l}"/>
+      </geometry>
       <origin xyz="0 0 0" rpy="0 ${PI_2} 0"/>
       <material name="red"/>
@@ -82,21 +97,6 @@
 			<origin xyz="0 0 0" rpy="0 ${PI_2} 0"/>
       <geometry>
-        <cylinder radius="${shoulder_pitch_r}" length="${shoulder_pitch_l}"/>
-      </geometry>
-    </collision>
-  </link>
-  <link name="${prefix}_shoulder_roll_cylinder">
-    <visual>
-      <geometry>
         <cylinder radius="${shoulder_roll_r}" length="${shoulder_roll_l}"/>
       </geometry>
-      <origin xyz="0 0 0" rpy="${PI_2} 0 0"/>
-      <material name="red"/>
-    </visual>
-    <collision>
-			<origin xyz="0 0 0" rpy="${PI_2} 0 0"/>
-      <geometry>
-        <cylinder radius="${shoulder_roll_r}" length="${shoulder_roll_l}"/>
-      </geometry>
     </collision>
   </link>
@@ -134,9 +134,9 @@
         <cylinder radius="${elbow_r}" length="${elbow_l}"/>
       </geometry>
-      <origin xyz="0 0 0" rpy="${PI_2} 0 0"/>
-      <material name="red"/>
-    </visual>
-    <collision>
-			<origin xyz="0 0 0" rpy="${PI_2} 0 0"/>
+      <origin xyz="0 0 0" rpy="0 ${PI_2} 0"/>
+      <material name="red"/>
+    </visual>
+    <collision>
+			<origin xyz="0 0 0" rpy="0 ${PI_2} 0"/>
       <geometry>
         <cylinder radius="${elbow_r}" length="${elbow_l}"/>

File: urdfs/torso/torso.urdf.xacro (robot description, xacro)
@@ -37,5 +37,5 @@
 			<visual>
 				<geometry>
-					<box size="${shoulder_w} ${shoulder_l} ${shoulder_h}"/>
+					<box size="${shoulder_l} ${shoulder_w} ${shoulder_h}"/>
 				</geometry>
 				<origin xyz="0 0 0"/>
@@ -44,5 +44,5 @@
 			<collision>
 				<geometry>
-					<box size="${shoulder_w} ${shoulder_l} ${shoulder_h}"/>
+					<box size="${shoulder_l} ${shoulder_w} ${shoulder_h}"/>
 				</geometry>
 			</collision>
